File: kicad/dongle-flash.kicad_pcb (KiCad board)
At the start: 4 copper layers, 15.2 x 24 mm, 6 parts, among them J1 Conn_01x10_Male, J2 Conn_01x10_Male, J3 Conn_01x04, J4 Conn_01x04, J5 Conn_01x04, U1 MX25R6435FM2xx0

Commit message: update kicad project
Parts:
- moved J5 3.85 mm to (144.9, 75.1), turned to 180 degrees
Routing:
- net +3V0: track 5.25 -> 7.64 mm
- net /P1.15: track 18.0 -> 15.6 mm
Changed lines of the file:
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@@
   )
   (footprint "Connector_JST:JST_SH_BM04B-SRSS-TB_1x04-1MP_P1.00mm_Vertical" (layer "F.Cu")
-    (at 141.07 75.72 -90)
+    (at 144.87 75.12 180)
     (descr "JST SH series connector, BM04B-SRSS-TB (http://www.jst-mfg.com/product/pdf/eng/eSH.pdf), generated with kicad-footprint-generator")
     (tags "connector JST SH side entry")
@@
     (property "Sheetname" "")
     (attr smd)
-    (fp_text reference "J5" (at 4.89 -1.95 -270) (layer "F.SilkS")
-      (effects (font (size 1 1) (thickness 0.15)))
-    )
-    (fp_text value "Conn_01x04" (at 14.5 -0.3 -270) (layer "F.Fab")
-      (effects (font (size 1 1) (thickness 0.15)))
-    )
-    (fp_text user "${REFERENCE}" (at 18.14 1.47 -270) (layer "F.Fab")
+    (fp_text reference "J5" (at 4.89 -1.95) (layer "F.SilkS")
+      (effects (font (size 1 1) (thickness 0.15)))
+    )
+    (fp_text value "Conn_01x04" (at 14.5 -0.3) (layer "F.Fab")
+      (effects (font (size 1 1) (thickness 0.15)))
+    )
+    (fp_text user "${REFERENCE}" (at 18.14 1.47) (layer "F.Fab")
       (effects (font (size 1 1) (thickness 0.15)))
     )
@@
     (fp_line (start -1.35 -1.55) (end -1.65 -1.55) (layer "F.Fab") (width 0.1))
     (fp_line (start -0.65 -1.55) (end -0.65 -0.95) (layer "F.Fab") (width 0.1))
-    (pad "1" smd roundrect (at -1.5 1.325 270) (size 0.6 1.55) (layers "F.Cu" "F.Paste" "F.Mask") (roundrect_rratio 0.25)
+    (pad "1" smd roundrect (at -1.5 1.325 180) (size 0.6 1.55) (layers "F.Cu" "F.Paste" "F.Mask") (roundrect_rratio 0.25)
       (net 16 "/P1.15") (pinfunction "Pin_1") (pintype "passive"))
-    (pad "2" smd roundrect (at -0.5 1.325 270) (size 0.6 1.55) (layers "F.Cu" "F.Paste" "F.Mask") (roundrect_rratio 0.25)
+    (pad "2" smd roundrect (at -0.5 1.325 180) (size 0.6 1.55) (layers "F.Cu" "F.Paste" "F.Mask") (roundrect_rratio 0.25)
       (net 15 "/P0.02") (pinfunction "Pin_2") (pintype "passive"))
-    (pad "3" smd roundrect (at 0.5 1.325 270) (size 0.6 1.55) (layers "F.Cu" "F.Paste" "F.Mask") (roundrect_rratio 0.25)
+    (pad "3" smd roundrect (at 0.5 1.325 180) (size 0.6 1.55) (layers "F.Cu" "F.Paste" "F.Mask") (roundrect_rratio 0.25)
       (net 12 "+3V0") (pinfunction "Pin_3") (pintype "passive"))
-    (pad "4" smd roundrect (at 1.5 1.325 270) (size 0.6 1.55) (layers "F.Cu" "F.Paste" "F.Mask") (roundrect_rratio 0.25)
+    (pad "4" smd roundrect (at 1.5 1.325 180) (size 0.6 1.55) (layers "F.Cu" "F.Paste" "F.Mask") (roundrect_rratio 0.25)
       (net 10 "GND") (pinfunction "Pin_4") (pintype "passive"))
-    (pad "MP" smd roundrect (at -2.8 -1.2 270) (size 1.2 1.8) (layers "F.Cu" "F.Paste" "F.Mask") (roundrect_rratio 0.2083333333))
-    (pad "MP" smd roundrect (at 2.8 -1.2 270) (size 1.2 1.8) (layers "F.Cu" "F.Paste" "F.Mask") (roundrect_rratio 0.2083333333))
+    (pad "MP" smd roundrect (at -2.8 -1.2 180) (size 1.2 1.8) (layers "F.Cu" "F.Paste" "F.Mask") (roundrect_rratio 0.2083333333))
+    (pad "MP" smd roundrect (at 2.8 -1.2 180) (size 1.2 1.8) (layers "F.Cu" "F.Paste" "F.Mask") (roundrect_rratio 0.2083333333))
     (model "${KICAD6_3DMODEL_DIR}/Connector_JST.3dshapes/JST_SH_BM04B-SRSS-TB_1x04-1MP_P1.00mm_Vertical.wrl"
       (offset (xyz 0 0 0))
@@
   (segment (start 146.4 85.19) (end 148.49 85.19) (width 0.25) (layer "F.Cu") (net 7))
   (segment (start 144.4 85.19) (end 144.4 84.54) (width 0.25) (layer "F.Cu") (net 12))
+  (segment (start 144.38 72.89) (end 143.33 71.84) (width 0.25) (layer "F.Cu") (net 12))
   (segment (start 144.37 78.65) (end 143.63 77.91) (width 0.25) (layer "F.Cu") (net 12))
+  (segment (start 144.38 73.795) (end 144.38 72.89) (width 0.25) (layer "F.Cu") (net 12))
   (segment (start 141.42 71.178) (end 140.97 71.628) (width 0.5) (layer "F.Cu") (net 12))
   (segment (start 141.42 70.23) (end 141.42 71.178) (width 0.5) (layer "F.Cu") (net 12))
@@
   (segment (start 137.315 78.585) (end 137.315 78.74) (width 0.25) (layer "In1.Cu") (net 15))
   (segment (start 146.38 73.795) (end 147.575 73.795) (width 0.25) (layer "F.Cu") (net 16))
-  (segment (start 144.38 72.89) (end 143.33 71.84) (width 0.25) (layer "F.Cu") (net 16))
-  (segment (start 144.38 73.795) (end 144.38 72.89) (width 0.25) (layer "F.Cu") (net 16))
   (segment (start 147.575 73.795) (end 147.6 73.77) (width 0.25) (layer "F.Cu") (net 16))
   (via (at 147.6 73.77) (size 0.8) (drill 0.4) (layers "F.Cu" "B.Cu") (net 16))
