File: kicad/dongle-flash.kicad_sch (KiCad schematic)
At the start: 6 parts, among them J1 Conn_01x10_Male, J2 Conn_01x10_Male, J3 Conn_01x04, J4 Conn_01x04, J5 Conn_01x04, U1 MX25R6435FM2xx0

Commit message: update kicad project
Connections:
- no-connect marks 3 -> 4
Changed lines of the file:
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@@
   (no_connect (at 102.87 102.87))
   (no_connect (at 102.87 100.33))
+  (no_connect (at 149.86 53.34))
   (wire (pts (xy 116.84 99.06) (xy 125.73 99.06))
     (stroke (width 0) (type default) (color 0 0 0 0))
